Commit message: Stable vision

File: iiwa_stack/iiwa_description/urdf/iiwa.gazebo.xacro (robot description, xacro)
@@ -1,4 +1,4 @@
 <?xml version="1.0"?>
-<robot xmlns:xacro="http://www.ros.org/wiki/xacro">
+<robot xmlns:xacro="http://ros.org/wiki/xacro">
   <xacro:macro name="iiwa_gazebo" params="side">
     <!-- Load Gazebo lib and set the robot namespace -->

File: iiwa_stack/iiwa_description/urdf/iiwa.transmission.xacro (robot description, xacro)
@@ -1,4 +1,4 @@
 <?xml version="1.0"?>
-<robot xmlns:xacro="http://www.ros.org/wiki/xacro">
+<robot xmlns:xacro="http://ros.org/wiki/xacro">
   <xacro:macro name="iiwa_transmission" params="hardware_interface side">
     <transmission name="${side}_tran_1">

File: iiwa_stack/iiwa_description/urdf/iiwa.urdf (robot description, URDF)
Before this commit: robot iiwa, 23 links, 22 joints
Links:
- removed link L_hand
- removed link L_link_0
- removed link L_link_1
- removed link L_link_2
- removed link L_link_3
- removed link L_link_4
- removed link L_link_5
- removed link L_link_6
- removed link L_link_7
- removed link L_link_ee
- removed link R_hand
- removed link body
- removed link desktop
- added link R_left_inner_finger, mass 0.0104003125914103; collision mesh filename=package://robotiq_2f_140_gripper_visualization/meshes/colli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; visual mesh filename=package://robotiq_2f_140_gripper_visualization/meshes/visua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
- added link R_left_inner_finger_pad; collision box size=0.03 0.07 0.0075; visual box size=0.027 0.065 0.0075
- added link R_left_inner_knuckle, mass 0.0271177346495152; collision mesh filename=package://robotiq_2f_140_gripper_visualization/meshes/colli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; visual mesh filename=package://robotiq_2f_140_gripper_visualization/meshes/visua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
- added link R_left_outer_finger, mass 0.022614240507152; collision mesh filename=package://robotiq_2f_140_gripper_visualization/meshes/colli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; visual mesh filename=package://robotiq_2f_140_gripper_visualization/meshes/visua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
- added link R_left_outer_knuckle, mass 0.00853198276973456; collision mesh filename=package://robotiq_2f_140_gripper_visualization/meshes/colli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; visual mesh filename=package://robotiq_2f_140_gripper_visualization/meshes/visua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
- added link R_right_inner_finger, mass 0.0104003125914103; collision mesh filename=package://robotiq_2f_140_gripper_visualization/meshes/colli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; visual mesh filename=package://robotiq_2f_140_gripper_visualization/meshes/visua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
- added link R_right_inner_finger_pad; collision box size=0.03 0.07 0.0075; visual box size=0.027 0.065 0.0075
- added link R_right_inner_knuckle, mass 0.0271177346495152; collision mesh filename=package://robotiq_2f_140_gripper_visualization/meshes/colli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; visual mesh filename=package://robotiq_2f_140_gripper_visualization/meshes/visua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
- added link R_right_outer_finger, mass 0.022614240507152; collision mesh filename=package://robotiq_2f_140_gripper_visualization/meshes/colli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; visual mesh filename=package://robotiq_2f_140_gripper_visualization/meshes/visua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
- added link R_right_outer_knuckle, mass 0.00853198276973456; collision mesh filename=package://robotiq_2f_140_gripper_visualization/meshes/colli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; visual mesh filename=package://robotiq_2f_140_gripper_visualization/meshes/visua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
- added link R_robotiq_arg2f_base_link, mass 0.22652; collision mesh filename=package://robotiq_2f_140_gripper_visualization/meshes/colli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; visual mesh filename=package://robotiq_2f_140_gripper_visualization/meshes/visua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
- added link camera_holder_link, mass 10; collision mesh filename=package://iiwa_description/meshes/base_part3_camera_holder_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; visual mesh filename=package://iiwa_description/meshes/base_part3_camera_holder.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
- added link cushion_link, mass 5; collision box size=1.1 1.6 0.068; visual box size=1.1 1.6 0.068
- added link lift_link, mass 47.592; collision mesh filename=package://iiwa_description/meshes/base_part1_lift.stl; visual mesh filename=package://iiwa_description/meshes/base_part1_lift.stl
- added link neck_link, mass 18.271; collision mesh filename=package://iiwa_description/meshes/base_part2_neck.stl; visual mesh filename=package://iiwa_description/meshes/base_part2_neck.stl
- added link reference_frame; visual sphere radius=0.01
- added link table_link, mass 1356.3; collision mesh filename=package://iiwa_description/meshes/base_part0_table_c.stl; visual mesh filename=package://iiwa_description/meshes/base_part0_table.stl
- link R_link_ee: mass 5 -> None; geometry 
Joints:
- removed joint L_hand_joint
- removed joint L_joint_1
- removed joint L_joint_2
- removed joint L_joint_3
- removed joint L_joint_4
- removed joint L_joint_5
- removed joint L_joint_6
- removed joint L_joint_7
- removed joint L_joint_ee
- removed joint R_hand_joint
- removed joint body_L_joint
- removed joint body_R_joint
- removed joint body_desktop_joint
- removed joint world_body_joint
- added joint R_finger_joint: type revolute, parent R_robotiq_arg2f_base_link, child R_left_outer_knuckle, origin xyz=0 -0.030601 0.054905 rpy=2.29579632679 0 0, axis -1 0 0, limit lower=0 upper=0.7 effort=1000 velocity=2.0
- added joint R_gripper_joint: type fixed, parent R_link_ee, child R_robotiq_arg2f_base_link, origin xyz=0 0 -0.214 rpy=0 0 1.57079632679
- added joint R_left_inner_finger_joint: type revolute, parent R_left_outer_finger, child R_left_inner_finger, origin xyz=0 0.0817554015893473 -0.0282203446692936 rpy=-0.725 0 0, axis 1 0 0, limit lower=-0.8757 upper=0.8757 effort=1000 velocity=2.0, mimic joint=R_finger_joint multiplier=1 offset=0
- added joint R_left_inner_finger_pad_joint: type fixed, parent R_left_inner_finger, child R_left_inner_finger_pad, origin xyz=0 0.0457554015893473 -0.0272203446692936 rpy=0 0 0, axis 0 0 1
- added joint R_left_inner_knuckle_joint: type revolute, parent R_robotiq_arg2f_base_link, child R_left_inner_knuckle, origin xyz=0 -0.0127 0.06142 rpy=2.29579632679 0 0.0, axis 1 0 0, limit lower=-0.8757 upper=0.8757 effort=1000 velocity=2.0, mimic joint=R_finger_joint multiplier=-1 offset=0
- added joint R_left_outer_finger_joint: type fixed, parent R_left_outer_knuckle, child R_left_outer_finger, origin xyz=0 0.01821998610742 0.0260018192872234 rpy=0 0 0, axis 1 0 0
- added joint R_right_inner_finger_joint: type revolute, parent R_right_outer_finger, child R_right_inner_finger, origin xyz=0 0.0817554015893473 -0.0282203446692936 rpy=-0.725 0 0, axis 1 0 0, limit lower=-0.8757 upper=0.8757 effort=1000 velocity=2.0, mimic joint=R_finger_joint multiplier=1 offset=0
- added joint R_right_inner_finger_pad_joint: type fixed, parent R_right_inner_finger, child R_right_inner_finger_pad, origin xyz=0 0.0457554015893473 -0.0272203446692936 rpy=0 0 0, axis 0 0 1
- added joint R_right_inner_knuckle_joint: type revolute, parent R_robotiq_arg2f_base_link, child R_right_inner_knuckle, origin xyz=0 0.0127 0.06142 rpy=2.29579632679 0 -3.14159265359, axis 1 0 0, limit lower=-0.8757 upper=0.8757 effort=1000 velocity=2.0, mimic joint=R_finger_joint multiplier=-1 offset=0
- added joint R_right_outer_finger_joint: type fixed, parent R_right_outer_knuckle, child R_right_outer_finger, origin xyz=0 0.01821998610742 0.0260018192872234 rpy=0 0 0, axis 1 0 0
- added joint R_right_outer_knuckle_joint: type revolute, parent R_robotiq_arg2f_base_link, child R_right_outer_knuckle, origin xyz=0 0.030601 0.054905 rpy=2.29579632679 0 3.14159265359, axis 1 0 0, limit lower=-0.725 upper=0.725 effort=1000 velocity=2.0, mimic joint=R_finger_joint multiplier=-1 offset=0
- added joint camera_holder_joint: type fixed, parent neck_link, child camera_holder_link, origin xyz=0 0 0.220 rpy=0 0 0
- added joint lift_neck_joint: type fixed, parent lift_link, child neck_link, origin xyz=-0.105 0 0.599 rpy=0 0 0, axis 0 0 1, limit lower=-0.7854 upper=0.7854 effort=300 velocity=1
- added joint neck_link_R_joint: type fixed, parent neck_link, child R_link_0, origin xyz=0.010 -0.158604 0.105 rpy=0 1.57079632679 -0.436332312999
- added joint reference_frame_joint: type fixed, parent cushion_link, child reference_frame, origin xyz=0 0 0.034 rpy=0 0 0
- added joint table_cushion_joint: type fixed, parent table_link, child cushion_link, origin xyz=0.95 0 1.0 rpy=0 0 0
- added joint table_lift_joint: type fixed, parent table_link, child lift_link, origin xyz=0.526 0 0.913 rpy=0 0 0, axis 0 0 1, limit lower=0 upper=0.450 effort=100 velocity=1.0
- added joint world_table_joint: type fixed, parent world, child table_link, origin xyz=0 0 0 rpy=0 0 0
- joint R_joint_ee: origin xyz=0 0 0.070 rpy=0 0 0 -> xyz=0 0 0.295 rpy=0 0 0

File: iiwa_stack/iiwa_description/urdf/iiwa.urdf.xacro (robot description, xacro)
@@ -1,4 +1,4 @@
 <?xml version="1.0"?>
-<robot name="iiwa" xmlns:xacro="http://www.ros.org/wiki/xacro">
+<robot name="iiwa" xmlns:xacro="http://ros.org/wiki/xacro">
   <!-- Import Rviz colors -->
   <xacro:include filename="$(find iiwa_description)/urdf/materials.xacro" />
@@ -11,78 +11,45 @@
   <xacro:arg name="hardware_interface" default="PositionJointInterface"/>
   <xacro:arg name="robot_name" default="iiwa"/>
-  <!--z = 0.458-->
-  <xacro:arg name="L_origin_xyz" default="0.153055 0.0595 0.758"/>
-  <xacro:arg name="L_origin_rpy" default="-1.0471975512 -1.5707963268 3.1415926536"/>
-  <xacro:arg name="R_origin_xyz" default="-0.153055 0.0595 0.758"/>
-  <xacro:arg name="R_origin_rpy" default="-1.0471975512 1.5707963268 3.1415926536"/>
+<xacro:arg name="L_origin_xyz" default="0.010 0.158604 0.105"/>
+<xacro:arg name="L_origin_rpy" default="0 ${PI/2} ${25*PI/180}"/>
+<xacro:arg name="R_origin_xyz" default="0.010 -0.158604 0.105"/>
+<xacro:arg name="R_origin_rpy" default="0 ${PI/2} ${-25*PI/180}"/>
   <!-- Fix to world just for testing -->
   <link name="world" />
-  <!--body-=======================================================================-->
-  <joint name="world_body_joint" type="fixed">
-    <origin xyz="0 0.297 0.92" rpy="0 0 0"/>
-      <parent link="world"/>
-      <child link="body"/>
+  <xacro:include filename="$(find iiwa_description)/urdf/platform.xacro"/>
+  <xacro:platform/>
+  <joint name="world_table_joint" type="fixed">
+    <origin xyz="0 0 0" rpy="0 0 0"/>
+    <parent link="world"/>
+    <child link="table_link"/>
   </joint>
-  <link name="body">
-      <inertial>
-        <origin xyz="0 0 0" rpy="0 0 0"/>
-        <mass value="5"/>
-        <inertia ixx="0.05"  ixy="0"  ixz="0" iyy="0.06" iyz="0" izz="0.03" />
-      </inertial>
-      <visual>
-        <!--<origin xyz="-0.6264 -1.0574 -0.92" rpy="0 0 0"/>-->
-        <origin xyz="0 0 0" rpy="0 0 0"/>
-        <geometry>
-          <mesh filename="package://iiwa_description/meshes/iiwa7/visual/body.stl"/>
-        </geometry>
-        <material name="White"/>
-      </visual>
-      <collision>
-        <origin xyz="0 0 0" rpy="0 0 0"/>
-        <geometry>
-          <mesh filename="package://iiwa_description/meshes/iiwa7/collision/body.stl"/>
-        </geometry>
-        <material name="White"/>
-      </collision>
-      </link>
-  <!--===========================================================================-->
+<!-- neck_link -->
   <!--iiwa-======================================================================-->
   <!--L_arm-->
-  <xacro:iiwa side="L" hardware_interface="$(arg hardware_interface)" parent="body">
+  <xacro:iiwa side="L" hardware_interface="$(arg hardware_interface)"  parent="neck_link" ee_z="${0.070 +0.225}">
     <origin xyz="$(arg L_origin_xyz)" rpy="$(arg L_origin_rpy)" />
   </xacro:iiwa>
   <!--R_arm-->
-  <xacro:iiwa side="R" hardware_interface="$(arg hardware_interface)" parent="body">
+  <xacro:iiwa side="R" hardware_interface="$(arg hardware_interface)"  parent="neck_link" ee_z="${0.070 +0.225}">
     <origin xyz="$(arg R_origin_xyz)" rpy="$(arg R_origin_rpy)" />
   </xacro:iiwa>
   <!--===========================================================================-->
-  <!--desktop-===================================================================-->
-  <joint name="body_desktop_joint" type="fixed">
-      <origin xyz="0 -0.6 0.034" rpy="0 0 0"/>
-      <parent link="body"/>
-      <child link="desktop"/>
+   <!--Import Robotiq gripper -->
+  <xacro:include filename="$(find robotiq_2f_140_gripper_visualization)/urdf/robotiq_arg2f_140_model_macro.xacro" />
+  <!--Left Robotiq gripper==-0.160-======================================================-->
+  <xacro:robotiq_arg2f_140 prefix="L_"/>
+  <joint name="L_gripper_joint" type="fixed">
+      <origin xyz="0 0 ${0.011-0.225}" rpy="0 0 ${PI/2}"/>
+      <parent link="L_link_ee"/>
+      <child link="L_robotiq_arg2f_base_link"/>
   </joint>
-  <link name="desktop">
-      <inertial>
-        <origin xyz="0 0 0" rpy="0 0 0"/>
-        <mass value="5"/>
-        <inertia ixx="0.05"  ixy="0"  ixz="0" iyy="0.06" iyz="0" izz="0.03" />
-      </inertial>
-      <visual>
-        <origin xyz=" 0 0 0" rpy="0 0 0" />
-        <geometry>
-          <box size="1.6 1.1 0.068"/>
-        </geometry>
-        <material name="White"/>
-      </visual>
-      <collision>
-        <origin xyz="0 0 0" rpy="0 0 0"/>
-        <geometry>
-          <box size="1.6 1.1 0.068"/>
-        </geometry>
-        <material name="White"/>
-      </collision>
-  </link>
-  <!--===========================================================================-->
+  <!--Right Robotiq gripper-====================================================-->
+  <xacro:robotiq_arg2f_140 prefix="R_"/>
+  <joint name="R_gripper_joint" type="fixed">
+      <origin xyz="0 0 ${0.011-0.225}" rpy="0 0 ${PI/2}"/>
+      <parent link="R_link_ee"/>
+      <child link="R_robotiq_arg2f_base_link"/>
+  </joint>
+  <!--=========================================================================-->
   <!-- Load Gazebo lib and set the robot namespace -->
     <gazebo>

File: iiwa_stack/iiwa_description/urdf/iiwa.xacro (robot description, xacro)
@@ -1,4 +1,4 @@
 <?xml version="1.0"?>
-<robot name="iiwa" xmlns:xacro="http://www.ros.org/wiki/xacro">
+<robot name="iiwa" xmlns:xacro="http://ros.org/wiki/xacro">
   <!-- Import all Gazebo-customization elements, including Gazebo colors -->
   <xacro:include filename="$(find iiwa_description)/urdf/iiwa.gazebo.xacro" />
@@ -13,5 +13,5 @@
   <xacro:property name="max_effort" value="300"/>
   <xacro:property name="max_velocity" value="10"/>
-  <xacro:macro name="iiwa" params="parent hardware_interface side *origin">
+  <xacro:macro name="iiwa" params="parent hardware_interface side *origin ee_z=0.07">
     <!--joint between {parent} and link_0-->
     <joint name="${parent}_${side}_joint" type="fixed">
@@ -289,53 +289,7 @@
       <parent link="${side}_link_7"/>
       <child link="${side}_link_ee"/>
-      <origin xyz="0 0 0.070" rpy="0 0 0"/>
-    </joint>
-    <link name="${side}_link_ee">
-      <inertial>
-        <origin xyz="0 0 0" rpy="0 0 0"/>
-        <mass value="5"/>
-        <inertia ixx="0.05"  ixy="0"  ixz="0" iyy="0.06" iyz="0" izz="0.03" />
-      </inertial>
-      <visual>
-        <origin xyz=" 0 0 0.06" rpy="0 0 0" />
-        <geometry>
-          <box size="0.085 0.095 0.17"/>
-        </geometry>
-        <material name="White"/>
-      </visual>
-      <collision>
-        <origin xyz="0 0 0.06" rpy="0 0 0"/>
-        <geometry>
-          <box size="0.085 0.095 0.17"/>
-        </geometry>
-        <material name="White"/>
-      </collision>
-    </link>
-    <joint name="${side}_hand_joint" type="fixed">
-      <origin xyz="0.03 0 0.345" rpy="0 0 0"/>
-      <parent link="${side}_link_ee"/>
-      <child link="${side}_hand"/>
-    </joint>
-    <link name="${side}_hand">
-      <inertial>
-        <origin xyz="0 0 0" rpy="0 0 0"/>
-        <mass value="5"/>
-        <inertia ixx="0.05"  ixy="0"  ixz="0" iyy="0.06" iyz="0" izz="0.03" />
-      </inertial>
-      <visual>
-        <origin xyz=" 0 0 -0.095" rpy="0 0 0" />
-        <geometry>
-          <box size="0.015 0.10 0.19"/>
-        </geometry>
-        <material name="White"/>
-      </visual>
-      <collision>
-        <origin xyz="0 0 -0.095" rpy="0 0 0"/>
-        <geometry>
-          <box size="0.015 0.10 0.19"/>
-        </geometry>
-        <material name="White"/>
-      </collision>
-    </link>
+      <origin xyz="0 0 ${ee_z}" rpy="0 0 0"/>
+    </joint>
+    <link name="${side}_link_ee"> </link>
     <!--Extensions -->
     <xacro:iiwa_gazebo side="${side}" />

File: iiwa_stack/iiwa_description/urdf/utilities.xacro (robot description, xacro)
@@ -1,4 +1,4 @@
 <?xml version="1.0"?>
-<robot xmlns:xacro="http://www.ros.org/wiki/xacro">
+<robot xmlns:xacro="http://ros.org/wiki/xacro">
   <xacro:property name="PI" value="3.1415926535897931"/>
 <!-- The following macros are adapted from the LWR 4 definitions of the RCPRG - https://github.com/RCPRG-ros-pkg/lwr_robot -->
